File: minimalist/squiggle-minimalist.kicad_pcb (KiCad board)
At the start: 2 copper layers, 235.1 x 115.3 mm, 71 parts, among them J1 02x05, J2 02x05, SW1 switch, SW10 switch, SW11 switch, SW12 switch, SW13 switch, SW14 switch, SW15 switch, SW16 switch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

Commit message: finished routing minimalist.
Parts:
- turned diode4 to 296.6 degrees
- turned diode8 to 296.6 degrees
Routing:
- net ROW0B: track 0.00 -> 259.5 mm
- net ROW1B: track 0.00 -> 236.1 mm
- net ROW2B: track 0.00 -> 212.1 mm
- net COL9: track 0.00 -> 182.7 mm
- net COL6: track 0.00 -> 157.3 mm
- net COL8: track 0.00 -> 156.8 mm
- net COL5: track 0.00 -> 136.9 mm
- net COL7: track 0.00 -> 135.6 mm
- net ROW3B: track 0.00 -> 66.2 mm
- net Net-(diode8-Pad2): track 0.00 -> 9.19 mm
- net Net-(diode4-Pad2): track 0.00 -> 8.70 mm
- net Net-(diode3-Pad2): track 0.00 -> 3.82 mm
- net Net-(diode17-Pad2): track 0.00 -> 3.82 mm
- net Net-(diode9-Pad2): track 0.00 -> 3.82 mm
- net Net-(diode7-Pad2): track 0.00 -> 3.82 mm
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- added copper zone on B.Cu, net (none)
- added copper zone on F.Cu, net (none)
Other:
- outline, holes or cut-outs redrawn

Commit message: added some new footprints.
Parts:
- added Ref**: Val**, footprints:hole-four, F.Cu at (140.0, 83.0)
- added Ref**: Val**, footprints:hole-four, F.Cu at (136.0, 83.0)
- added Ref**: Val**, footprints:hole-four, F.Cu at (140.0, 67.5)
- added Ref**: Val**, footprints:hole-four, F.Cu at (136.0, 67.5)
- added Ref**: Val**, footprints:hole-four, F.Cu at (136.0, 50.0)
- added Ref**: Val**, footprints:hole-four, F.Cu at (140.0, 50.0)
- added Ref**: Val**, footprints:hole-four, F.Cu at (140.0, 35.5)
- added Ref**: Val**, footprints:hole-four, F.Cu at (136.0, 35.5)
- moved J2 1.00 mm to (148.2, 70.0)
- moved diode1 1.00 mm to (177.0, 30.0)
- moved diode10 1.00 mm to (215.0, 40.0)
- moved diode11 1.00 mm to (215.0, 59.0)
- moved diode12 1.00 mm to (234.0, 27.0)
- moved diode13 1.00 mm to (234.0, 46.0)
- moved diode14 1.00 mm to (234.0, 65.0)
- moved diode15 1.00 mm to (253.0, 39.0)
- moved diode16 1.00 mm to (253.0, 58.0)
- moved diode17 1.00 mm to (253.0, 77.0)
- moved diode2 1.00 mm to (177.0, 49.0)
- moved diode3 1.00 mm to (177.0, 68.0)
- moved diode4 1.00 mm to (169.2, 103.2)
- moved diode5 1.00 mm to (196.0, 28.0)
- moved diode6 1.00 mm to (196.0, 47.0)
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Other:
- board size 235.1 x 115.3 mm -> 236.1 x 115.3 mm
